File: 01_Schematic/Multi_Tone.kicad_sch (KiCad schematic)
At the start: 65 parts, among them J1 PW_INPUT, J2 PW_OUTPUT, J3 SIGNAL_INPUT, Q1 2N3904, Q2 2N3904, Q3 2N3904, U1 LM2904, U2 LM2902, U3 L7812, U4 L7912

Commit message: Finishd PCB design
Parts:
- BR1:  Manufacturer (none) -> DigiKey; MPN (none) -> DB107-BPMS-ND; Notes (none) -> Link r https://www.digikey.co.uk/en/products/detail/mcc-mic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
- C1, C3:  Manufacturer (none) -> RS; MPN (none) -> 703-7318; Notes (none) -> https://uk.rs-online.com/web/p/aluminium-capacitors/7037318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
- C10:  Manufacturer (none) -> RS; MPN (none) -> 133-5725; Notes (none) -> https://uk.rs-online.com/web/p/mlccs-multilayer-ceramic-cap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
- C11, C12, C13, C14, C5, C6, C7, C8:  Manufacturer (none) -> RS; MPN (none) -> 852-3270; Notes (none) -> https://uk.rs-online.com/web/p/mlccs-multilayer-ceramic-cap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
- C2, C4:  Manufacturer (none) -> RS; MPN (none) -> 526-1597; Notes (none) -> https://uk.rs-online.com/web/p/aluminium-capacitors/5261597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
- C9:  Manufacturer (none) -> RS; MPN (none) -> 841-0733; Notes (none) -> https://uk.rs-online.com/web/p/mlccs-multilayer-ceramic-cap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
- D1: value LED Y -> LEDY;  Manufacturer (none) -> DigiKey; MPN (none) -> 5962-XL-302UYD-ND; Notes (none) -> https://www.digikey.co.uk/en/products/detail/xinglight/XL-3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
- D2:  Manufacturer (none) -> DigiKey; MPN (none) -> 5962-XL-302URD-ND; Notes (none) -> https://www.digikey.co.uk/en/products/detail/xinglight/XL-3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
- D3, D5, D7:  Manufacturer (none) -> Digikey; MPN (none) -> 1N4148FS-ND; Notes (none) -> https://www.digikey.co.uk/en/products/detail/onsemi/1N4148/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
- D4:  Manufacturer (none) -> DigiKey; MPN (none) -> 5962-XL-302UBD-ND; Notes (none) -> https://www.digikey.co.uk/en/products/detail/xinglight/XL-3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
- D6:  Manufacturer (none) -> DigiKey; MPN (none) -> 5962-XL-302UGD-ND; Notes (none) -> https://www.digikey.co.uk/en/products/detail/xinglight/XL-3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
- J1, J2:  Manufacturer (none) -> RS; MPN (none) -> 790-1092; Notes (none) -> https://uk.rs-online.com/web/p/pcb-terminal-blocks/7901092
- J3:  Manufacturer (none) -> RS; MPN (none) -> 790-1098; Notes (none) -> https://uk.rs-online.com/web/p/pcb-terminal-blocks/7901098
- Q1, Q2, Q3:  Manufacturer (none) -> RS; MPN (none) -> 843-1575; Notes (none) -> https://uk.rs-online.com/web/p/bipolar-transistors/8431575?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
- R1:  Manufacturer (none) -> RS; MPN (none) -> 125-1159; Notes (none) -> https://uk.rs-online.com/web/p/through-hole-resistors/12511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
- R10, R3, R7:  Manufacturer (none) -> RS; MPN (none) -> 755-1233; Notes (none) -> https://uk.rs-online.com/web/p/surface-mount-resistors/7551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
- R11, R15:  Manufacturer (none) -> RS; MPN (none) -> 148-893; Notes (none) -> https://uk.rs-online.com/web/p/through-hole-resistors/01488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
- R12, R8:  Manufacturer (none) -> RS; MPN (none) -> 124-2864; Notes (none) -> https://uk.rs-online.com/web/p/through-hole-resistors/12428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
- R13:  Manufacturer (none) -> RS; MPN (none) -> 683-3575; Notes (none) -> https://uk.rs-online.com/web/p/through-hole-resistors/68335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
- R14, R4, R9:  Manufacturer (none) -> RS; MPN (none) -> 224-0424P; Notes (none) -> https://uk.rs-online.com/web/p/surface-mount-resistors/2240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
- R16:  Manufacturer (none) -> RS; MPN (none) -> 487-7141; Notes (none) -> https://uk.rs-online.com/web/p/through-hole-resistors/48771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
- R2:  Manufacturer (none) -> RS; MPN (none) -> 683-6552; Notes (none) -> https://uk.rs-online.com/web/p/surface-mount-resistors/6836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
- R5, R6:  Manufacturer (none) -> RS; MPN (none) -> 683-3099P; Notes (none) -> https://uk.rs-online.com/web/p/through-hole-resistors/68330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
- RV1:  Manufacturer (none) -> RS; MPN (none) -> 167-3364; Notes (none) -> https://uk.rs-online.com/web/p/trimmer-potentiometers/16733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
- TP1, TP10, TP11, TP12, TP13, TP14, TP15, TP16, TP2, TP3, TP4, TP5, TP6, TP7, TP8, TP9:  Manufacturer (none) -> DigiKey; MPN (none) -> 2057-PH1-01-UA-ND; Notes (none) -> https://www.digikey.co.uk/en/products/detail/adam-tech/PH1-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
- U1:  Manufacturer (none) -> RS; MPN (none) -> 121-8467; Notes (none) -> https://uk.rs-online.com/web/p/op-amps/1218467?gb=s
- U2:  Manufacturer (none) -> RS; MPN (none) -> 121-9109; Notes (none) -> https://uk.rs-online.com/web/p/op-amps/1219109?gb=s
- U3:  Manufacturer (none) -> RS; MPN (none) -> 918-1975; Notes (none) -> https://uk.rs-online.com/web/p/voltage-regulators/9181975?g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
- U4:  Manufacturer (none) -> RS; MPN (none) -> 168-6803; Notes (none) -> https://uk.rs-online.com/web/p/voltage-regulators/1686803?g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
Other:
- note added: "DECOUPLING CAPS"
