File: 02_PCB/Multi_Tone.kicad_pcb (KiCad board)
At the start: 2 copper layers, 100 x 80 mm, 65 parts, among them J1 PW_INPUT, J2 PW_OUTPUT, J3 SIGNAL_INPUT, Q1 2N3904, Q2 2N3904, Q3 2N3904, U1 LM2904, U2 LM2902, U3 L7812, U4 L7912

Commit message: Finishd PCB design
Parts:
- moved TP15 63.5 mm to (69.8, 33.0)
- moved U3 39.1 mm to (55.8, 22.3), turned to 90 degrees
- moved C5 5.09 mm to (72.2, 71.8)
- moved R7 4.54 mm to (98.2, 82.8)
- moved R10 4.54 mm to (98.2, 58.5)
- moved R3 4.51 mm to (98.2, 33.2)
- moved TP14 3.00 mm to (31.0, 81.8)
- moved RV1 1.39 mm to (68.0, 38.0)
- moved C11 1.17 mm to (66.0, 76.0)
- moved D4 0.96 mm to (107.2, 77.0)
- moved C2 0.79 mm to (29.8, 44.2)
- moved C4 0.75 mm to (29.5, 35.2)
- moved D2 0.75 mm to (107.5, 27.5)
- moved D6 0.68 mm to (107.8, 53.0)
- moved U4 0.51 mm to (48.5, 42.0)
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Connections:
- net Net-(J1-Pin_1) renamed /VAC+
- net Net-(J1-Pin_3) renamed /VAC-
Routing:
- net +12V: track 38.9 -> 231.6 mm, vias 0 -> 2
- net /SIGNAL: track 0.00 -> 92.3 mm
- net /V_AMP: track 0.00 -> 90.8 mm
- net /OUT_LOW: track 0.00 -> 64.8 mm, vias 0 -> 2
- net -12V: track 50.8 -> 112.0 mm, vias 0 -> 1
- net /OUT_HIGH: track 0.00 -> 59.4 mm
- net /OUT_MID: track 0.00 -> 40.4 mm
- net Net-(U2C-+): track 0.00 -> 21.9 mm, vias 0 -> 1
- net Net-(C10-Pad1): track 0.00 -> 20.7 mm
- net Net-(Q2-B): track 0.00 -> 17.0 mm
- net Net-(Q1-B): track 0.00 -> 16.5 mm
- net Net-(Q3-B): track 0.00 -> 16.2 mm
- net Net-(C5-Pad2): track 0.00 -> 15.8 mm
- net Net-(BR1-+): track 6.77 -> 20.9 mm
- net Net-(D4-A): track 0.00 -> 12.4 mm
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- removed copper zone on F.Cu, net GND
Other:
- board text added: "+12V"
- board text added: "-12V"
- board text added: "BASE_HIGH"
- board text added: "BASE_LOW"
- board text added: "BASE_MID"
- board text added: "GND"
- board text added: "OUT_HIGH"
- board text added: "OUT_LOW"
- board text added: "OUT_MID"
- board text added: "OUT_SIG"
- board text added: "SIGNAL"
- board text added: "VAC+"
- board text added: "VAC-"
- board text added: "V_AMP"
